Commit message: optimize topic load and reduce no of topic

File: zed_wrapper/urdf/zed_macro.urdf.xacro (robot description, xacro)
@@ -1,5 +1,5 @@
 <?xml version="1.0"?>
 <!--
-// Copyright 2025 Stereolabs
+// Copyright 2024 Stereolabs
 //
 // Licensed under the Apache License, Version 2.0 (the "License");
@@ -70,13 +70,4 @@
       <xacro:property name="mono" value="false" />
     </xacro:if>
-    <xacro:if value="${model == 'zedxhdr'}">
-      <xacro:property name="baseline" value="0.12" />
-      <xacro:property name="height" value="0.032" />
-      <xacro:property name="bottom_slope" value="0.0" />
-      <xacro:property name="screw_offset_x" value="0.0" />
-      <xacro:property name="screw_offset_z" value="-0.016" />
-      <xacro:property name="optical_offset_x" value="-0.01" />
-      <xacro:property name="mono" value="false" />
-    </xacro:if>
     <xacro:if value="${model == 'zedxm'}">
       <xacro:property name="baseline" value="0.05" />
@@ -88,22 +79,4 @@
       <xacro:property name="mono" value="false" />
     </xacro:if>
-    <xacro:if value="${model == 'zedxhdrmini'}">
-      <xacro:property name="baseline" value="0.05" />
-      <xacro:property name="height" value="0.032" />
-      <xacro:property name="bottom_slope" value="0.0" />
-      <xacro:property name="screw_offset_x" value="0.0" />
-      <xacro:property name="screw_offset_z" value="-0.016" />
-      <xacro:property name="optical_offset_x" value="-0.01" />
-      <xacro:property name="mono" value="false" />
-    </xacro:if>
-    <xacro:if value="${model == 'zedxhdrmax'}">
-      <xacro:property name="baseline" value="0.170" />
-      <xacro:property name="height" value="0.032" />
-      <xacro:property name="bottom_slope" value="0.0" />
-      <xacro:property name="screw_offset_x" value="0.0" />
-      <xacro:property name="screw_offset_z" value="-0.016" />
-      <xacro:property name="optical_offset_x" value="-0.01" />
-      <xacro:property name="mono" value="false" />
-    </xacro:if>
     <xacro:if value="${model == 'virtual'}">
       <xacro:property name="baseline" value="${custom_baseline}" />
@@ -133,15 +106,6 @@
       <xacro:property name="mono" value="true" />
     </xacro:if>
-    <xacro:if value="${model == 'zedxonehdr'}">
-      <xacro:property name="baseline" value="0.0" />
-      <xacro:property name="height" value="0.025" />
-      <xacro:property name="bottom_slope" value="0.0" />
-      <xacro:property name="screw_offset_x" value="0.00" />
-      <xacro:property name="screw_offset_z" value="-0.0125" />
-      <xacro:property name="optical_offset_x" value="0.0" />
-      <xacro:property name="mono" value="true" />
-    </xacro:if>
     <!-- Camera mounting point (the threaded screw hole in the bottom) -->
-    <link name="${name}_camera_link" />
+    <link name="base_link" />
     <!-- Camera Center -->
     <link name="${name}_camera_center">
@@ -150,5 +114,5 @@
           <origin xyz="${screw_offset_x} 0 ${screw_offset_z}" rpy="0 0 0"/>
           <geometry>
-            <mesh filename="file://$(find zed_msgs)/meshes/${model}.stl"/>
+<mesh filename="file://$(find zed_msgs)/meshes/${model}.stl"/>
           </geometry>
           <material name="${model}_mat" />
@@ -157,5 +121,5 @@
           <origin xyz="${screw_offset_x} 0 ${screw_offset_z}" rpy="0 0 0"/>
           <geometry>
-            <mesh filename="file://$(find zed_msgs)/meshes/${model}.stl"/>
+<mesh filename="file://$(find zed_msgs)/meshes/${model}.stl"/>
           </geometry>
         </collision>
@@ -163,5 +127,5 @@
     </link>
     <joint name="${name}_camera_center_joint" type="fixed">
-      <parent link="${name}_camera_link"/>
+      <parent link="base_link"/>
       <child link="${name}_camera_center"/>
       <origin xyz="0 0 ${height/2}" rpy="0 ${bottom_slope} 0" />
@@ -174,5 +138,5 @@
             <origin xyz="0 0 0" rpy="0 0 0"/>
             <geometry>
-              <mesh filename="file://$(find zed_msgs)/meshes/${model}.stl"/>
+  <mesh filename="file://$(find zed_msgs)/meshes/${model}.stl"/>
             </geometry>
             <material name="${model}_mat" />
@@ -181,5 +145,5 @@
             <origin xyz="0 0 0" rpy="0 0 0"/>
             <geometry>
-              <mesh filename="file://$(find zed_msgs)/meshes/${model}.stl"/>
+  <mesh filename="file://$(find zed_msgs)/meshes/${model}.stl"/>
             </geometry>
           </collision>
@@ -203,5 +167,5 @@
             <origin xyz="0 0 0" rpy="0 0 0"/>
             <geometry>
-              <mesh filename="file://$(find zed_msgs)/meshes/${model}.stl"/>
+  <mesh filename="file://$(find zed_msgs)/meshes/${model}.stl"/>
             </geometry>
             <material name="${model}_mat" />
@@ -210,5 +174,5 @@
             <origin xyz="0 0 0" rpy="0 0 0"/>
             <geometry>
-              <mesh filename="file://$(find zed_msgs)/meshes/${model}.stl"/>
+  <mesh filename="file://$(find zed_msgs)/meshes/${model}.stl"/>
             </geometry>
           </collision>
