Commit message: added domain_bridge_config,changes in urdf

File: zed_wrapper/urdf/zed_descr.urdf.xacro (robot description, xacro)
@@ -24,7 +24,13 @@
   <xacro:arg name="gnss_y" default="0.0" />
   <xacro:arg name="gnss_z" default="0.0" />
+  <link name="base_link"/>
   <xacro:include filename="$(find zed_wrapper)/urdf/zed_macro.urdf.xacro" />
   <xacro:zed_camera name="$(arg camera_name)" model="$(arg camera_model)" custom_baseline="$(arg custom_baseline)" enable_gnss="$(arg enable_gnss)">
 	    <origin xyz="$(arg gnss_x) $(arg gnss_y) $(arg gnss_z)" rpy="0 0 0"/>
   </xacro:zed_camera>
+  <joint name="$(arg camera_name)_mount_joint" type="fixed">
+    <parent link="base_link"/>
+    <child link="$(arg camera_name)_camera_link"/>
+    <origin xyz="0 0 0" rpy="0 0 0"/>
+  </joint>
 </robot>

File: zed_wrapper/urdf/zed_macro.urdf.xacro (robot description, xacro)
@@ -107,5 +107,6 @@
     </xacro:if>
     <!-- Camera mounting point (the threaded screw hole in the bottom) -->
-    <link name="base_link" />
+    <!-- <link name="base_link" /> -->
+    <link name="${name}_camera_link" />
     <!-- Camera Center -->
     <link name="${name}_camera_center">
@@ -127,5 +128,5 @@
     </link>
     <joint name="${name}_camera_center_joint" type="fixed">
-      <parent link="base_link"/>
+      <parent link="${name}_camera_link"/>
       <child link="${name}_camera_center"/>
       <origin xyz="0 0 ${height/2}" rpy="0 ${bottom_slope} 0" />
