Commit message: Fix TF listener QoS and restore ZED URDF

File: zed_wrapper/urdf/zed_descr.urdf.xacro (robot description, xacro)
@@ -24,13 +24,7 @@
   <xacro:arg name="gnss_y" default="0.0" />
   <xacro:arg name="gnss_z" default="0.0" />
-  <link name="base_link"/>
   <xacro:include filename="$(find zed_wrapper)/urdf/zed_macro.urdf.xacro" />
   <xacro:zed_camera name="$(arg camera_name)" model="$(arg camera_model)" custom_baseline="$(arg custom_baseline)" enable_gnss="$(arg enable_gnss)">
 	    <origin xyz="$(arg gnss_x) $(arg gnss_y) $(arg gnss_z)" rpy="0 0 0"/>
   </xacro:zed_camera>
-  <joint name="$(arg camera_name)_mount_joint" type="fixed">
-    <parent link="base_link"/>
-    <child link="$(arg camera_name)_camera_link"/>
-    <origin xyz="0 0 0" rpy="0 0 0"/>
-  </joint>
 </robot>

Commit message: Wrap official ZED description with base link mount

File: zed_wrapper/urdf/zed_descr.urdf.xacro (robot description, xacro)
@@ -24,7 +24,13 @@
   <xacro:arg name="gnss_y" default="0.0" />
   <xacro:arg name="gnss_z" default="0.0" />
-  <xacro:include filename="$(find zed_wrapper)/urdf/zed_macro.urdf.xacro" />
+  <xacro:include filename="$(find zed_description)/urdf/zed_macro.urdf.xacro" />
+  <link name="base_link"/>
   <xacro:zed_camera name="$(arg camera_name)" model="$(arg camera_model)" custom_baseline="$(arg custom_baseline)" enable_gnss="$(arg enable_gnss)">
 	    <origin xyz="$(arg gnss_x) $(arg gnss_y) $(arg gnss_z)" rpy="0 0 0"/>
   </xacro:zed_camera>
+  <joint name="$(arg camera_name)_mount_joint" type="fixed">
+    <parent link="base_link"/>
+    <child link="$(arg camera_name)_camera_link"/>
+    <origin xyz="0 0 0" rpy="0 0 0"/>
+  </joint>
 </robot>
